Commit message: feat: 更新地图

File: robot_yang/src/carlike_robot_description/xacro/car_description.xacro (robot description, xacro)
@@ -8,3 +8,10 @@
     <!-- <xacro:include filename="$(find carlike_robot_description)/xacro/sensors/lidar.xacro" /> -->
     <xacro:include filename="$(find carlike_robot_description)/xacro/sensors/VLP-16.xacro" />
+    <gazebo reference="base_footprint">
+      <visual>
+        <plugin filename="libdraw_traj.so" name="drawtrajPlugin">
+          <topicName>/odom</topicName>
+        </plugin>
+      </visual>
+    </gazebo>
 </robot>
